File: MASA Antenna Control Board.kicad_pcb (KiCad board)
At the start: 2 copper layers, 80 x 59.2 mm, 32 parts, among them J1 UJ2-MBH-1-SMT, J2 Conn_01x06_Male, J3 Conn_01x02_Male, J4 Conn_01x02_Male, J5 Conn_01x04_Male, U1 BL654PA, U2 XBP9B-DPST-001, U3 XBP9B-DPST-001, U4 XBP9B-DPST-001, U5 TPS563200

Commit message: Finished routing
Parts:
- added J6: 1-1123723-2, Tracking-Antenna-Control-Board:TE_1-1123723-2, F.Cu at (134.7, 42.9)
- added J7: 1-1123723-2, Tracking-Antenna-Control-Board:TE_1-1123723-2, F.Cu at (193.9, 18.7)
- added J8: 1-1123723-2, Tracking-Antenna-Control-Board:TE_1-1123723-2, F.Cu at (203.9, 18.8)
- moved C4 69.9 mm to (159.0, 53.6), turned to 180 degrees
- moved R3 66.1 mm to (163.2, 53.6), turned to 180 degrees
- moved C3 51.5 mm to (153.0, 41.7)
- moved R2 51.2 mm to (156.0, 42.8)
- moved R1 39.1 mm to (149.9, 40.0)
- moved C2 35.6 mm to (153.5, 38.6), turned to 270 degrees
- moved J1 19.8 mm to (216.7, 19.9)
- moved C13 4.99 mm to (223.4, 85.3), turned to 90 degrees
Connections:
- U1 pad 11: Net-(U1-Pad11) -> StepperFour
- U1 pad 13: Net-(U1-Pad13) -> StepperThree
- U1 pad 7: Net-(U1-Pad7) -> StepperTwo
- U1 pad 9: Net-(U1-Pad9) -> StepperOne
Routing:
- net RSSI3: track 128.4 -> 22.6 mm
- net Net-(R2-Pad1): track 4.12 -> 100.6 mm
- net RSSI1: track 102.1 -> 27.9 mm
- net Net-(R3-Pad1): track 5.09 -> 65.8 mm
- net +3V3: track 137.0 -> 188.9 mm, vias 2 -> 3
- net RSSI2: track 61.5 -> 18.0 mm, vias 2 -> 0
- net Net-(R1-Pad1): track 4.46 -> 47.3 mm, vias 0 -> 2
- net StepperThree: track 0.00 -> 38.1 mm
- net StepperFour: track 0.00 -> 33.9 mm
- net StepperOne: track 0.00 -> 27.7 mm
- net StepperTwo: track 0.00 -> 23.3 mm
- net D-: track 30.5 -> 50.2 mm
- net USB_VBUS: track 37.8 -> 57.5 mm
- net D+: track 29.4 -> 49.1 mm
- net GND: track 34.5 -> 43.0 mm, vias 13 -> 15
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Other:
- board size 80 x 59.2 mm -> 95.3 x 90.7 mm
